Commit message: reflect changes from 14.07

File: amr_description/xacro/back_lidar.xacro (robot description, xacro)
@@ -1,11 +1,11 @@
 <?xml version="1.0"?>
 <robot xmlns:xacro="http://www.ros.org/wiki/xacro">
-    <joint name="back_lidar_joint" type="fixed">
-        <origin xyz="-0.770 0.3675 0.085" rpy="0 0 2.355" />    <!-- <origin xyz="-0.770 0.3675 0.085" rpy="0 0 3.14159265359" /> -->
+    <joint name="back_laser_joint" type="fixed">
+        <origin xyz="-0.685 0.360 0.085" rpy="0 3.14 -0.785" />    <!-- <origin xyz="-0.770 0.3675 0.085" rpy="0 0 3.14159265359" /> -->
         <parent link="base_link" />
-        <child link="back_lidar_link" />
+        <child link="back_laser_link" />
         <axis xyz="0 0 1" />
     </joint>
-    <link name="back_lidar_link">
+    <link name="back_laser_link">
         <visual>
             <origin xyz="0 0 0" rpy="0 0 0" />
@@ -29,6 +29,6 @@
         </inertial>
     </link>
-    <gazebo reference="back_lidar_link">
-        <sensor type="ray" name="back_lidar_sensor">
+    <gazebo reference="back_laser_link">
+        <sensor type="ray" name="back_laser_sensor">
             <pose>0 0 0 0 0 0</pose>
             <visualize>false</visualize>
@@ -56,5 +56,5 @@
             <plugin name="gazebo_ros_head_rplidar_controller" filename="libgazebo_ros_laser.so">
                 <topicName>/scan_back_laser</topicName>
-                <frameName>back_lidar_link</frameName>
+                <frameName>back_laser_link</frameName>
             </plugin>
         </sensor>

File: amr_description/xacro/front_lidar.xacro (robot description, xacro)
@@ -1,11 +1,11 @@
 <?xml version="1.0"?>
 <robot xmlns:xacro="http://www.ros.org/wiki/xacro" >
-    <joint name="front_lidar_joint" type="fixed">
-        <origin xyz="0.6225 -0.375 0.085" rpy="0 0 -0.785"/>
+    <joint name="front_laser_joint" type="fixed">
+        <origin xyz="0.70 -0.360 0.085" rpy="0 3.14 2.355"/>
         <parent link="base_link"/>
-        <child link="front_lidar_link"/>
+        <child link="front_laser_link"/>
         <axis xyz="0 0 1"/>
     </joint>
-    <link name="front_lidar_link">
+    <link name="front_laser_link">
         <visual>
             <origin xyz="0 0 0" rpy="0 0 0"/>
@@ -29,6 +29,6 @@
         </inertial>
     </link>
-    <gazebo reference="front_lidar_link">
-        <sensor type="ray" name="front_lidar_sensor">
+    <gazebo reference="front_laser_link">
+        <sensor type="ray" name="front_laser_sensor">
             <pose>0 0 0 0 0 0</pose>
             <visualize>false</visualize>
@@ -56,5 +56,5 @@
             <plugin name="gazebo_ros_head_rplidar_controller" filename="libgazebo_ros_laser.so">
                 <topicName>/scan_front_laser</topicName>
-                <frameName>front_lidar_link</frameName>
+                <frameName>front_laser_link</frameName>
             </plugin>
         </sensor>

File: amr_description/xacro/imu.xacro (robot description, xacro)
@@ -4,5 +4,5 @@
         <parent link="base_link" />
         <child link="imu_link" />
-        <origin xyz="-0.65 -0.005 0.008" rpy="0 0 -1.57" />
+        <origin xyz="-0.61 -0.005 0.105" rpy="0 3.14 0" />
     </joint>
     <link name="imu_link">

File: amr_description/xacro/left_wheel.xacro (robot description, xacro)
@@ -13,5 +13,5 @@
     <xacro:property name="left_wheel_Izz" value="0.021" />
     <joint name="left_wheel_joint" type="continuous">
-        <origin xyz="-0.074 0.315 -0.05" rpy="0 0 0" />
+        <origin xyz="0 0.315 -0.05" rpy="0 0 0" />
         <parent link="base_link" />
         <child link="left_wheel_link" />

File: amr_description/xacro/main.xacro (robot description, xacro)
@@ -10,9 +10,9 @@
 	</xacro:unless>
 	<xacro:include filename="$(find amr_description)/xacro/common_properties.xacro" />
-	<xacro:include filename="$(find amr_description)/xacro/gazebo.xacro" />
+	<!-- <xacro:include filename="$(find amr_description)/xacro/gazebo.xacro" /> -->
 	<xacro:include filename="$(find amr_description)/xacro/base_footprint.xacro" />
 	<xacro:include filename="$(find amr_description)/xacro/base.xacro" />
-	<xacro:include filename="$(find amr_description)/xacro/lift.xacro" />
-	<xacro:include filename="$(find amr_description)/xacro/caster_wheels.xacro" />
+	<!-- <xacro:include filename="$(find amr_description)/xacro/lift.xacro" /> -->
+	<!-- <xacro:include filename="$(find amr_description)/xacro/caster_wheels.xacro" /> -->
 	<xacro:include filename="$(find amr_description)/xacro/right_wheel.xacro" />
 	<xacro:include filename="$(find amr_description)/xacro/left_wheel.xacro" />

File: amr_description/xacro/right_wheel.xacro (robot description, xacro)
@@ -13,5 +13,5 @@
     <xacro:property name="right_wheel_Izz" value="0.021" />
     <joint name="right_wheel_joint" type="continuous">
-        <origin xyz="-0.074 -0.323 -0.05" rpy="0 0 0" />
+        <origin xyz="0 -0.315 -0.05" rpy="0 0 0" />
         <parent link="base_link" />
         <child link="right_wheel_link" />
